File: pcb/micromouse/micromouse.sch (EAGLE design)
At the start: 57 parts, among them J1 Connector_M1, J2 Connector_M1, J4 Programmer

Commit message: initial putting components in place
Parts:
- removed R1: 62, rcl:R-EU_R0805
- added LED3: Spacing_LED_front, led:LED5MM
- J2: value Connector_M1 -> Connector_M2
- LED4: value Front_wheel -> Spacing_LED_back
Connections:
- removed net N$2: LED4.A, R1.1
- net +3V3: no longer R1.2
- net GND: no longer LED4.C
Other:
- moved on the sheet: C20
Changed lines of the file:
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@@
 <part name="+3V4" library="supply1" library_urn="urn:adsk.eagle:library:371" deviceset="+3V3" device=""/>
 <part name="J1" library="con-ml" library_urn="urn:adsk.eagle:library:164" deviceset="ML6" device="" package3d_urn="urn:adsk.eagle:package:8675/1" value="Connector_M1"/>
-<part name="J2" library="con-ml" library_urn="urn:adsk.eagle:library:164" deviceset="ML6" device="" package3d_urn="urn:adsk.eagle:package:8675/1" value="Connector_M1"/>
+<part name="J2" library="con-ml" library_urn="urn:adsk.eagle:library:164" deviceset="ML6" device="" package3d_urn="urn:adsk.eagle:package:8675/1" value="Connector_M2"/>
 <part name="HC05/06" library="con-lsta" library_urn="urn:adsk.eagle:library:161" deviceset="FE06-1" device="" package3d_urn="urn:adsk.eagle:package:8191/1" value="UART"/>
 <part name="J4" library="con-lstb" library_urn="urn:adsk.eagle:library:162" deviceset="MA06-1" device="" package3d_urn="urn:adsk.eagle:package:8340/1" value="Programmer"/>
@@
 <part name="+9V" library="holes" library_urn="urn:adsk.eagle:library:237" deviceset="MOUNT-PAD-ROUND" device="3.0" package3d_urn="urn:adsk.eagle:package:14280/1" value="Battery"/>
 <part name="-" library="holes" library_urn="urn:adsk.eagle:library:237" deviceset="MOUNT-PAD-ROUND" device="3.0" package3d_urn="urn:adsk.eagle:package:14280/1" value="Battery"/>
-<part name="LED4" library="led" library_urn="urn:adsk.eagle:library:259" deviceset="LED" device="5MM" package3d_urn="urn:adsk.eagle:package:15799/2" value="Front_wheel"/>
+<part name="LED4" library="led" library_urn="urn:adsk.eagle:library:259" deviceset="LED" device="5MM" package3d_urn="urn:adsk.eagle:package:15799/2" value="Spacing_LED_back"/>
 <part name="+3V10" library="supply1" library_urn="urn:adsk.eagle:library:371" deviceset="+3V3" device=""/>
 <part name="+3V11" library="supply1" library_urn="urn:adsk.eagle:library:371" deviceset="+3V3" device=""/>
@@
 <part name="SV4" library="con-lstb" library_urn="urn:adsk.eagle:library:162" deviceset="MA10-2" device="" package3d_urn="urn:adsk.eagle:package:8331/1" value="Pin header"/>
 <part name="GND8" library="supply1" library_urn="urn:adsk.eagle:library:371" deviceset="GND" device=""/>
-<part name="R1" library="rcl" library_urn="urn:adsk.eagle:library:334" deviceset="R-EU_" device="R0805" package3d_urn="urn:adsk.eagle:package:23553/2" value="62"/>
-<part name="GND12" library="supply1" library_urn="urn:adsk.eagle:library:371" deviceset="GND" device=""/>
-<part name="+3V12" library="supply1" library_urn="urn:adsk.eagle:library:371" deviceset="+3V3" device=""/>
 <part name="C18" library="rcl" library_urn="urn:adsk.eagle:library:334" deviceset="C-EU" device="C0805" package3d_urn="urn:adsk.eagle:package:23617/2" value="100nF"/>
 <part name="GND25" library="supply1" library_urn="urn:adsk.eagle:library:371" deviceset="GND" device=""/>
@@
 <part name="L3" library="Eagle_WE-PD (rev20a)" deviceset="WE-PD_1210" device="" package3d_urn="urn:adsk.eagle:package:13009201/2" technology="_7447709331" value="330uH"/>
 <part name="L1" library="Eagle_WE-PD (rev20a)" deviceset="WE-PD_1210" device="" package3d_urn="urn:adsk.eagle:package:13009201/2" technology="_7447709331" value="330uH"/>
+<part name="LED3" library="led" library_urn="urn:adsk.eagle:library:259" deviceset="LED" device="5MM" package3d_urn="urn:adsk.eagle:package:15799/2" value="Spacing_LED_front"/>
+<part name="GND12" library="supply1" library_urn="urn:adsk.eagle:library:371" deviceset="GND" device=""/>
 </parts>
 <sheets>
@@
 <attribute name="VALUE" x="-68.58" y="185.42" size="1.778" layer="96"/>
 </instance>
-<instance part="R1" gate="G$1" x="-129.54" y="233.68" smashed="yes" rot="R90">
-<attribute name="NAME" x="-131.0386" y="229.87" size="1.778" layer="95" rot="R90"/>
-<attribute name="VALUE" x="-126.238" y="229.87" size="1.778" layer="96" rot="R90"/>
-</instance>
-<instance part="GND12" gate="1" x="-129.54" y="205.74" smashed="yes">
-<attribute name="VALUE" x="-132.08" y="203.2" size="1.778" layer="96"/>
-</instance>
-<instance part="+3V12" gate="G$1" x="-129.54" y="248.92" smashed="yes">
-<attribute name="VALUE" x="-129.54" y="241.3" size="1.778" layer="96" rot="R90"/>
-</instance>
 <instance part="C18" gate="G$1" x="104.14" y="200.66" smashed="yes" rot="R180">
 <attribute name="NAME" x="102.616" y="200.279" size="1.778" layer="95" rot="R180"/>
@@
 <attribute name="VALUE" x="294.64" y="25.4" size="1.778" layer="96"/>
 </instance>
-<instance part="C20" gate="G$1" x="284.48" y="35.56" smashed="yes" rot="R180">
-<attribute name="NAME" x="290.576" y="35.179" size="1.778" layer="95" rot="R180"/>
-<attribute name="VALUE" x="293.116" y="40.259" size="1.778" layer="96" rot="R180"/>
+<instance part="C20" gate="G$1" x="284.48" y="60.96" smashed="yes" rot="R180">
+<attribute name="NAME" x="290.576" y="60.579" size="1.778" layer="95" rot="R180"/>
+<attribute name="VALUE" x="293.116" y="65.659" size="1.778" layer="96" rot="R180"/>
 </instance>
 <instance part="S1" gate="G$1" x="-81.28" y="347.98" smashed="yes" rot="R90">
@@
 <attribute name="NAME" x="10.16" y="294.64" size="1.27" layer="95" align="bottom-center"/>
 <attribute name="VALUE" x="6.35" y="289.56" size="1.27" layer="96"/>
+</instance>
+<instance part="LED3" gate="G$1" x="-144.78" y="218.44" smashed="yes">
+<attribute name="NAME" x="-141.224" y="213.868" size="1.778" layer="95" rot="R90"/>
+<attribute name="VALUE" x="-139.065" y="213.868" size="1.778" layer="96" rot="R90"/>
+</instance>
+<instance part="GND12" gate="1" x="284.48" y="55.88" smashed="yes">
+<attribute name="VALUE" x="281.94" y="53.34" size="1.778" layer="96"/>
 </instance>
 </instances>
@@
 </segment>
 <segment>
-<pinref part="LED4" gate="G$1" pin="C"/>
-<pinref part="GND12" gate="1" pin="GND"/>
-<wire x1="-129.54" y1="213.36" x2="-129.54" y2="208.28" width="0.1524" layer="91"/>
-</segment>
-<segment>
 <pinref part="C19" gate="G$1" pin="1"/>
 <wire x1="297.18" y1="33.02" x2="297.18" y2="30.48" width="0.1524" layer="91"/>
 <pinref part="GND26" gate="1" pin="GND"/>
+</segment>
+<segment>
 <pinref part="C20" gate="G$1" pin="1"/>
-<wire x1="284.48" y1="33.02" x2="297.18" y2="33.02" width="0.1524" layer="91"/>
-<junction x="297.18" y="33.02"/>
+<pinref part="GND12" gate="1" pin="GND"/>
 </segment>
 </net>
@@
 <wire x1="284.48" y1="68.58" x2="284.48" y2="73.66" width="0.1524" layer="91"/>
 <pinref part="C20" gate="G$1" pin="2"/>
-<wire x1="284.48" y1="40.64" x2="284.48" y2="68.58" width="0.1524" layer="91"/>
+<wire x1="284.48" y1="66.04" x2="284.48" y2="68.58" width="0.1524" layer="91"/>
 <junction x="284.48" y="68.58"/>
 </segment>
@@
 <pinref part="R10" gate="G$1" pin="2"/>
 <wire x1="218.44" y1="274.32" x2="218.44" y2="269.24" width="0.1524" layer="91"/>
-</segment>
-<segment>
-<pinref part="R1" gate="G$1" pin="2"/>
-<wire x1="-129.54" y1="238.76" x2="-129.54" y2="246.38" width="0.1524" layer="91"/>
-<pinref part="+3V12" gate="G$1" pin="+3V3"/>
 </segment>
 </net>
@@
 </segment>
 </net>
-<net name="N$2" class="0">
-<segment>
-<pinref part="R1" gate="G$1" pin="1"/>
-<pinref part="LED4" gate="G$1" pin="A"/>
-<wire x1="-129.54" y1="228.6" x2="-129.54" y2="220.98" width="0.1524" layer="91"/>
-</segment>
-</net>

Commit message: Exchanged 100 uF capacitors at voltage regulator to have 1210 mounting layout + added ground planes
Parts:
- C12, C14: device rcl:C-EUC0805 -> rcl:C-EUC1210
Changed lines of the file:
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@@
 <part name="RESET" library="switch-omron" library_urn="urn:adsk.eagle:library:377" deviceset="10-XX" device="" package3d_urn="urn:adsk.eagle:package:27496/1" value="B3F-1000"/>
 <part name="LM2575-5.0WU-(TR)" library="national-semiconductor" library_urn="urn:adsk.eagle:library:307" deviceset="LM2596" device="S" package3d_urn="urn:adsk.eagle:package:16438/2"/>
-<part name="C12" library="rcl" library_urn="urn:adsk.eagle:library:334" deviceset="C-EU" device="C0805" package3d_urn="urn:adsk.eagle:package:23617/2" value="100uF"/>
+<part name="C12" library="rcl" library_urn="urn:adsk.eagle:library:334" deviceset="C-EU" device="C1210" package3d_urn="urn:adsk.eagle:package:23619/2" value="100uF"/>
 <part name="C13" library="rcl" library_urn="urn:adsk.eagle:library:334" deviceset="C-EU" device="C0805" package3d_urn="urn:adsk.eagle:package:23617/2" value="330uF"/>
 <part name="D9" library="diode" library_urn="urn:adsk.eagle:library:210" deviceset="BAT19" device="" package3d_urn="urn:adsk.eagle:package:43344/2" value="1N5822"/>
@@
 <part name="P+3" library="supply1" library_urn="urn:adsk.eagle:library:371" deviceset="+5V" device=""/>
 <part name="LM2575-3.3WU-(TR)" library="national-semiconductor" library_urn="urn:adsk.eagle:library:307" deviceset="LM2596" device="S" package3d_urn="urn:adsk.eagle:package:16438/2"/>
-<part name="C14" library="rcl" library_urn="urn:adsk.eagle:library:334" deviceset="C-EU" device="C0805" package3d_urn="urn:adsk.eagle:package:23617/2" value="100uF"/>
+<part name="C14" library="rcl" library_urn="urn:adsk.eagle:library:334" deviceset="C-EU" device="C1210" package3d_urn="urn:adsk.eagle:package:23619/2" value="100uF"/>
 <part name="C15" library="rcl" library_urn="urn:adsk.eagle:library:334" deviceset="C-EU" device="C0805" package3d_urn="urn:adsk.eagle:package:23617/2" value="330uF"/>
 <part name="D10" library="diode" library_urn="urn:adsk.eagle:library:210" deviceset="BAT19" device="" package3d_urn="urn:adsk.eagle:package:43344/2" value="1N5822"/>
